File: Slepet.kicad_pcb (KiCad board)
At the start: 2 copper layers, 150.9 x 105 mm, 50 parts, among them J1 Conn_02x05_Odd_Even, U1 promicro

Commit message: ok
Parts:
- removed the HS1 at (80.2, -46.2)
- added HS2: Heatsink, footprints:baldy_luv_u, B.Cu at (74.5, -45.0)
- added HS3: Heatsink, footprints:baldy_luv_u, F.Cu at (212.3, -45.0)
- added HS4: Heatsink, footprints:baldy_luv_u, B.Cu at (212.3, -45.0)
- added HS5: Heatsink, footprints:hole-three, F.Cu at (145.9, -24.3)
- added HS6: Heatsink, footprints:hole-three, F.Cu at (140.7, -23.4)
- added HS7: Heatsink, footprints:hole-three, F.Cu at (151.5, -3.43)
- added HS8: Heatsink, footprints:hole-three, F.Cu at (135.3, -3.52)
- added J2: Conn_02x05_Odd_Even, footprints:connector-shrouded, F.Cu at (154.2, -16.5)
- added diode24: diode, footprints:diode, F.Cu at (157.7, -62.4)
- added diode25: diode, footprints:diode, F.Cu at (179.4, -68.0)
- added diode26: diode, footprints:diode, F.Cu at (201.5, -72.6)
- added diode27: diode, footprints:diode, F.Cu at (223.8, -75.9)
- added diode28: diode, footprints:diode, F.Cu at (246.8, -65.7)
- added diode29: diode, footprints:diode, F.Cu at (269.7, -66.7)
- added diode30: diode, footprints:diode, F.Cu at (162.7, -44.0)
- added diode31: diode, footprints:diode, F.Cu at (183.3, -49.4)
- added diode32: diode, footprints:diode, F.Cu at (204.4, -53.7)
- added diode33: diode, footprints:diode, F.Cu at (225.7, -57.0)
- added diode34: diode, footprints:diode, F.Cu at (247.8, -46.6)
- added diode35: diode, footprints:diode, F.Cu at (269.3, -47.6)
- added diode36: diode, footprints:diode, F.Cu at (167.6, -25.6)
- added diode37: diode, footprints:diode, F.Cu at (187.3, -30.8)
- added diode38: diode, footprints:diode, F.Cu at (207.4, -34.9)
- added diode39: diode, footprints:diode, F.Cu at (227.7, -38.0)
- added diode40: diode, footprints:diode, F.Cu at (248.8, -27.6)
- added diode41: diode, footprints:diode, F.Cu at (269.3, -28.6)
- added diode42: diode, footprints:diode, F.Cu at (154.8, 8.64)
- added diode43: diode, footprints:diode, F.Cu at (172.3, -1.19)
- added diode44: diode, footprints:diode, F.Cu at (190.7, -9.15)
- added diode45: diode, footprints:diode, F.Cu at (209.9, -15.1)
- added diode46: diode, footprints:diode, F.Cu at (229.7, -19.1)
- added switch24: switch, footprints:100-minimal, F.Cu at (165.4, -64.5)
- added switch25: switch, footprints:100-minimal, F.Cu at (187.2, -69.7)
- added switch26: switch, footprints:100-minimal, F.Cu at (209.4, -73.8)
- added switch27: switch, footprints:100-minimal, F.Cu at (231.7, -76.7)
- added switch28: switch, footprints:100-minimal, F.Cu at (254.8, -66.1)
- added switch29: switch, footprints:100-minimal, F.Cu at (277.3, -66.7)
- added switch30: switch, footprints:100-minimal, F.Cu at (170.4, -46.1)
- added switch31: switch, footprints:100-minimal, F.Cu at (191.2, -51.1)
- added switch32: switch, footprints:100-minimal, F.Cu at (212.3, -55.0)
- added switch33: switch, footprints:100-minimal, F.Cu at (233.7, -57.8)
- added switch34: switch, footprints:100-minimal, F.Cu at (255.8, -47.1)
- added switch35: switch, footprints:100-minimal, F.Cu at (277.3, -47.6)
- added switch36: switch, footprints:100-minimal, F.Cu at (175.3, -27.7)
- added switch37: switch, footprints:100-minimal, F.Cu at (195.1, -32.4)
- added switch38: switch, footprints:100-minimal, F.Cu at (215.3, -36.2)
- added switch39: switch, footprints:100-minimal, F.Cu at (235.7, -38.9)
- added switch40: switch, footprints:100-minimal, F.Cu at (256.8, -28.0)
- added switch41: switch, footprints:100-minimal, F.Cu at (277.3, -28.6)
- added switch42: switch, footprints:100-minimal, F.Cu at (161.7, 4.64)
- added switch43: switch, footprints:100-minimal, F.Cu at (179.6, -4.45)
- added switch44: switch, footprints:100-minimal, F.Cu at (198.3, -11.6)
- added switch45: switch, footprints:100-minimal, F.Cu at (217.8, -16.8)
- added switch46: switch, footprints:100-minimal, F.Cu at (237.7, -19.9)
- moved HS1 5.71 mm to (74.5, -45.0)
- moved U1 5.40 mm to (138.5, -51.1)
- moved J1 2.73 mm to (132.8, -16.5)
- moved diode12 2.07 mm to (124.4, -44.0)
- moved diode18 2.07 mm to (119.5, -25.5)
- moved diode6 2.07 mm to (129.3, -62.4)
- moved diode17 1.68 mm to (99.6, -30.8)
- moved diode11 1.68 mm to (103.6, -49.4)
- moved diode5 1.68 mm to (107.5, -68.0)
- moved diode21 1.56 mm to (96.0, -9.11), turned to 342 degrees
- moved diode10 1.28 mm to (82.5, -53.7)
- moved diode16 1.28 mm to (79.5, -34.9)
- moved diode4 1.28 mm to (85.4, -72.6)
- moved diode22 0.99 mm to (114.5, -1.17)
- moved diode19 0.90 mm to (57.2, -19.1)
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Connections:
- J1 pad 1: (no net) -> CL6
- J1 pad 10: (no net) -> CL1
- J1 pad 2: (no net) -> R8
- J1 pad 3: (no net) -> CL5
- J1 pad 4: (no net) -> R7
- J1 pad 5: (no net) -> CL4
- J1 pad 6: (no net) -> R6
- J1 pad 7: (no net) -> CL3
- J1 pad 8: (no net) -> R5
- J1 pad 9: (no net) -> CL2
- U1 pad 10: (no net) -> CL4
- U1 pad 11: (no net) -> CL5
- U1 pad 12: (no net) -> CL6
- U1 pad 13: (no net) -> R8
- U1 pad 14: (no net) -> R7
- U1 pad 15: (no net) -> R6
- U1 pad 16: (no net) -> R5
- U1 pad 17: (no net) -> RL4
- U1 pad 18: (no net) -> RL3
- U1 pad 19: (no net) -> RL2
- U1 pad 20: (no net) -> RL1
- U1 pad 7: (no net) -> CL1
- U1 pad 8: (no net) -> CL2
- U1 pad 9: (no net) -> CL3
- diode1 pad 1: Net-(diode1-Pad1) -> RL1
- diode10 pad 1: Net-(diode10-Pad1) -> RL2
- diode11 pad 1: Net-(diode10-Pad1) -> RL2
- diode12 pad 1: Net-(diode10-Pad1) -> RL2
- diode13 pad 1: Net-(diode13-Pad1) -> RL3
- diode14 pad 1: Net-(diode13-Pad1) -> RL3
- diode15 pad 1: Net-(diode13-Pad1) -> RL3
- diode16 pad 1: Net-(diode13-Pad1) -> RL3
- diode17 pad 1: Net-(diode13-Pad1) -> RL3
- diode18 pad 1: Net-(diode13-Pad1) -> RL3
- diode19 pad 1: Net-(diode19-Pad1) -> RL4
- diode2 pad 1: Net-(diode1-Pad1) -> RL1
- diode20 pad 1: Net-(diode19-Pad1) -> RL4
- diode21 pad 1: Net-(diode19-Pad1) -> RL4
- diode22 pad 1: Net-(diode19-Pad1) -> RL4
- diode23 pad 1: Net-(diode19-Pad1) -> RL4
- diode3 pad 1: Net-(diode1-Pad1) -> RL1
- diode4 pad 1: Net-(diode1-Pad1) -> RL1
- diode5 pad 1: Net-(diode1-Pad1) -> RL1
- diode6 pad 1: Net-(diode1-Pad1) -> RL1
- diode7 pad 1: Net-(diode10-Pad1) -> RL2
- diode8 pad 1: Net-(diode10-Pad1) -> RL2
- diode9 pad 1: Net-(diode10-Pad1) -> RL2
- switch1 pad 1: Net-(diode1-Pad2) -> CL1
- switch1 pad 2: Net-(switch1-Pad2) -> Net-(diode1-Pad2)
- switch10 pad 1: Net-(diode10-Pad2) -> CL4
- switch10 pad 2: Net-(switch10-Pad2) -> Net-(diode10-Pad2)
- switch11 pad 1: Net-(diode11-Pad2) -> CL5
- switch11 pad 2: Net-(switch11-Pad2) -> Net-(diode11-Pad2)
- switch12 pad 1: Net-(diode12-Pad2) -> CL6
- switch12 pad 2: Net-(switch12-Pad2) -> Net-(diode12-Pad2)
- switch13 pad 1: Net-(diode13-Pad2) -> CL1
- switch13 pad 2: Net-(switch1-Pad2) -> Net-(diode13-Pad2)
- switch14 pad 1: Net-(diode14-Pad2) -> CL2
- switch14 pad 2: Net-(switch14-Pad2) -> Net-(diode14-Pad2)
- switch15 pad 1: Net-(diode15-Pad2) -> CL3
- switch15 pad 2: Net-(switch15-Pad2) -> Net-(diode15-Pad2)
- switch16 pad 1: Net-(diode16-Pad2) -> CL4
- switch16 pad 2: Net-(switch10-Pad2) -> Net-(diode16-Pad2)
- switch17 pad 1: Net-(diode17-Pad2) -> CL5
- switch17 pad 2: Net-(switch11-Pad2) -> Net-(diode17-Pad2)
- switch18 pad 1: Net-(diode18-Pad2) -> CL6
- switch18 pad 2: Net-(switch12-Pad2) -> Net-(diode18-Pad2)
- switch19 pad 1: Net-(diode19-Pad2) -> CL2
- switch19 pad 2: Net-(switch14-Pad2) -> Net-(diode19-Pad2)
- switch2 pad 1: Net-(diode2-Pad2) -> CL2
- switch2 pad 2: Net-(switch14-Pad2) -> Net-(diode2-Pad2)
- switch20 pad 1: Net-(diode20-Pad2) -> CL3
- switch20 pad 2: Net-(switch15-Pad2) -> Net-(diode20-Pad2)
- switch21 pad 1: Net-(diode21-Pad2) -> CL4
- switch21 pad 2: Net-(switch10-Pad2) -> Net-(diode21-Pad2)
- switch22 pad 1: Net-(diode22-Pad2) -> CL5
- switch22 pad 2: Net-(switch11-Pad2) -> Net-(diode22-Pad2)
- switch23 pad 1: Net-(diode23-Pad2) -> CL6
- switch23 pad 2: Net-(switch12-Pad2) -> Net-(diode23-Pad2)
- switch3 pad 1: Net-(diode3-Pad2) -> CL3
- switch3 pad 2: Net-(switch15-Pad2) -> Net-(diode3-Pad2)
- switch4 pad 1: Net-(diode4-Pad2) -> CL4
- switch4 pad 2: Net-(switch10-Pad2) -> Net-(diode4-Pad2)
- switch5 pad 1: Net-(diode5-Pad2) -> CL5
- switch5 pad 2: Net-(switch11-Pad2) -> Net-(diode5-Pad2)
- switch6 pad 1: Net-(diode6-Pad2) -> CL6
- switch6 pad 2: Net-(switch12-Pad2) -> Net-(diode6-Pad2)
- switch7 pad 1: Net-(diode7-Pad2) -> CL1
- switch7 pad 2: Net-(switch1-Pad2) -> Net-(diode7-Pad2)
- switch8 pad 1: Net-(diode8-Pad2) -> CL2
- switch8 pad 2: Net-(switch14-Pad2) -> Net-(diode8-Pad2)
- switch9 pad 1: Net-(diode9-Pad2) -> CL3
- switch9 pad 2: Net-(switch15-Pad2) -> Net-(diode9-Pad2)
Routing:
- net CL1: track 0.00 -> 246.6 mm
- net CL2: track 0.00 -> 241.3 mm
- net CR1: track 0.00 -> 213.0 mm
- net CL3: track 0.00 -> 209.7 mm
- net RR1: track 0.00 -> 186.8 mm
- net CR2: track 0.00 -> 186.2 mm
- net CL4: track 0.00 -> 183.3 mm
- net CR3: track 0.00 -> 165.2 mm
- net RL4: track 0.00 -> 162.0 mm
- net CL5: track 0.00 -> 159.1 mm
- net RR2: track 0.00 -> 158.3 mm
- net RL3: track 0.00 -> 149.4 mm
- net CR4: track 0.00 -> 141.4 mm
- net RL2: track 0.00 -> 135.3 mm
- net CL6: track 0.00 -> 133.1 mm
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- added copper zone on B.Cu, net (none)
- added copper zone on F.Cu, net (none)
Other:
- board size 150.9 x 105 mm -> 286.9 x 105 mm

Commit message: sneaky
Connections:
- J2 pad 10: CR1 -> CL1
- switch29 pad 2: CR1 -> CL1
- switch35 pad 2: CR1 -> CL1
- switch41 pad 2: CR1 -> CL1
Routing:
- net CL1: track 246.6 -> 494.7 mm
- net CR1: track 213.0 -> 0.00 mm

Commit message: to lessen the burden.
Parts:
- switch1, switch10, switch11, switch12, switch13, switch14, switch15, switch16, switch17, switch18, switch19, switch2, switch20, switch21, switch22, switch23, switch24, switch25, switch26, switch27, switch28, switch29, switch3, switch30, switch31, switch32, switch33, switch34, switch35, switch36, switch37, switch38, switch39, switch4, switch40, switch41, switch42, switch43, switch44, switch45, switch46, switch5, switch6, switch7, switch8, switch9: footprint footprints:100-minimal -> rick-kicad-footprints:100-minimal-no-3d
