File: Slepet.sch (KiCad schematic (older format))
At the start: 49 parts, among them J1 Conn_02x05_Odd_Even, U1 promicro

Commit message: ok
Parts:
- added HS2, HS3, HS4: Heatsink, footprints:baldy_luv_u, symbol mechanical:Heatsink
- added HS5, HS6, HS7, HS8: Heatsink, footprints:hole-three, symbol mechanical:Heatsink
- added J2: Conn_02x05_Odd_Even, footprints:connector-shrouded, symbol Connector_Generic:Conn_02x05_Odd_Even
- added diode24, diode25, diode26, diode27, diode28, diode29, diode30, diode31, diode32, diode33, diode34, diode35, diode36, diode37, diode38, diode39, diode40, diode41, diode42, diode43, diode44, diode45, diode46: diode, footprints:diode, symbol rick-kicad-lib:diode
- added switch24, switch25, switch26, switch27, switch28, switch29, switch30, switch31, switch32, switch33, switch34, switch35, switch36, switch37, switch38, switch39, switch40, switch41, switch42, switch43, switch44, switch45, switch46: switch, footprints:100-minimal, symbol rick-kicad-lib:switch
Connections:
- net labels added: CL1, CL2, CL3, CL4, CL5, CL6, CR1, CR2, CR3, CR4, CR5, CR6, R5, R6, R7, R8, RL1, RL2, RL3, RL4, RR1, RR2, RR3, RR4
- wire segments 46 -> 92
Other:
- moved on the sheet: switch1, switch10, switch11, switch12, switch13, switch14, switch15, switch16, switch17, switch18, switch19, switch2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

Commit message: sneaky
Connections:
- net CR1 is gone; now on net CL1: J2.10 (Pin_10), switch29.2, switch35.2, switch41.2
Changed lines of the file:
@@
 Text GLabel 10075 1900 2    50   Input ~ 0
 RR4
-Text GLabel 1950 7075 3    50   Input ~ 0
-CR6
 Text GLabel 2800 7075 3    50   Input ~ 0
 CR5
@@
 CR2
 Text GLabel 6200 7075 3    50   Input ~ 0
-CR1
+CL1
 Text GLabel 9575 2100 0    50   Input ~ 0
 CR4
@@
 Text GLabel 9575 2000 0    50   Input ~ 0
 CR5
+Text GLabel 10075 2300 2    50   Input ~ 0
+CL1
+Text GLabel 1950 7075 3    50   Input ~ 0
+CR6
 Text GLabel 9575 1900 0    50   Input ~ 0
 CR6
-Text GLabel 10075 2300 2    50   Input ~ 0
-CR1
 $EndSCHEMATC

Commit message: to lessen the burden.
Parts:
- switch1, switch10, switch11, switch12, switch13, switch14, switch15, switch16, switch17, switch18, switch19, switch2, switch20, switch21, switch22, switch23, switch24, switch25, switch26, switch27, switch28, switch29, switch3, switch30, switch31, switch32, switch33, switch34, switch35, switch36, switch37, switch38, switch39, switch4, switch40, switch41, switch42, switch43, switch44, switch45, switch46, switch5, switch6, switch7, switch8, switch9: footprint footprints:100-minimal -> rick-kicad-footprints:100-minimal-no-3d
